File: schematic/_saved_badge.sch (KiCad schematic (older format))
At the start: 36 parts, among them J1 Left2, J10 Left1, J2 Left3, J3 Bottom, J4 Serial, J5 Pennies, J6 Right1, J7 Right2, J8 Right3, J9 Right4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

Commit message: Finished v1 schematic
Parts:
- removed J5: Pennies, symbol Conn_01x04
- added J11: Penny2, Wire_Pads:Penny, symbol Conn_01x01
- added J12: Penny1, Wire_Pads:Penny, symbol Conn_01x01
- added J13: Penny0, Wire_Pads:Penny, symbol Conn_01x01
- added J14: Power, Wire_Pads:SolderWirePad_2x_1mmDrill, symbol Conn_01x02
- added J15: Right5, Connectors:GS2, symbol Conn_01x02
- added J5: Penny3, Wire_Pads:Penny, symbol Conn_01x01
- J1: footprint (none) -> Wire_Pads:SolderWirePad_4xInline_1mmDrill
- J10: footprint (none) -> Connectors:GS2
- J2, J4, J6: footprint (none) -> Wire_Pads:SolderWirePad_2x_1mmDrill
- J7, J9: footprint (none) -> Wire_Pads:SolderWirePad_single_1mmDrill
Connections:
- net GND: no longer C11.2, U1.1 (GND), U1.15 (GND), U1.38 (GND), U1.39 (GND-PAD)
- net IO16: now also J15.2 (Pin_2)
- net IO17: now also J15.1 (Pin_1)
- net P0: now also J13.1 (Pin_1)
- net P1: now also J12.1 (Pin_1)
- net P2: now also U1.13 (IO14), J11.1 (Pin_1)
- net P3: now also J5.1 (Pin_1); no longer U1.13 (IO14)
- net VDD: now also J14.1 (Pin_1)
- net VSS: now also C11.2, U1.1 (GND), U1.15 (GND), U1.38 (GND), U1.39 (GND-PAD), J14.2 (Pin_2)
Other:
- moved on the sheet: J3
Changed lines of the file:
@@
 Wire Wire Line
 	7800 5050 7650 5050
-$Comp
-L GND #PWR04
-U 1 1 5AD68DB2
-P 7650 5050
-F 0 "#PWR04" H 7650 4800 50  0001 C CNN
-F 1 "GND" H 7650 4900 50  0000 C CNN
-F 2 "" H 7650 5050 50  0001 C CNN
-F 3 "" H 7650 5050 50  0001 C CNN
-	1    7650 5050
-	0    1    1    0
-$EndComp
 Wire Wire Line
 	9650 4900 9800 4900
@@
 Wire Wire Line
 	9650 5000 9900 5000
-$Comp
-L GND #PWR05
-U 1 1 5AD68EC5
-P 9900 5000
-F 0 "#PWR05" H 9900 4750 50  0001 C CNN
-F 1 "GND" H 9900 4850 50  0000 C CNN
-F 2 "" H 9900 5000 50  0001 C CNN
-F 3 "" H 9900 5000 50  0001 C CNN
-	1    9900 5000
-	0    -1   -1   0
-$EndComp
 Wire Wire Line
 	8300 5400 8300 5500
-$Comp
-L GND #PWR06
-U 1 1 5AD6937B
-P 8300 5500
-F 0 "#PWR06" H 8300 5250 50  0001 C CNN
-F 1 "GND" H 8300 5350 50  0000 C CNN
-F 2 "" H 8300 5500 50  0001 C CNN
-F 3 "" H 8300 5500 50  0001 C CNN
-	1    8300 5500
-	1    0    0    -1
-$EndComp
 Wire Wire Line
 	7800 3750 7550 3750
@@
 	7550 3750 7550 3350
 $Comp
-L VDD #PWR07
+L VDD #PWR04
 U 1 1 5AD69713
 P 7550 3350
-F 0 "#PWR07" H 7550 3200 50  0001 C CNN
+F 0 "#PWR04" H 7550 3200 50  0001 C CNN
 F 1 "VDD" H 7550 3500 50  0000 C CNN
 F 2 "" H 7550 3350 50  0001 C CNN
@@
 Connection ~ 7050 3500
 $Comp
-L GND #PWR08
+L GND #PWR05
 U 1 1 5AD69A65
 P 6950 3500
-F 0 "#PWR08" H 6950 3250 50  0001 C CNN
+F 0 "#PWR05" H 6950 3250 50  0001 C CNN
 F 1 "GND" H 6950 3350 50  0000 C CNN
 F 2 "" H 6950 3500 50  0001 C CNN
@@
 	6650 3400 6650 3300
 $Comp
-L VDD #PWR09
+L VDD #PWR06
 U 1 1 5AD69EC1
 P 6650 3300
-F 0 "#PWR09" H 6650 3150 50  0001 C CNN
+F 0 "#PWR06" H 6650 3150 50  0001 C CNN
 F 1 "VDD" H 6650 3450 50  0000 C CNN
 F 2 "" H 6650 3300 50  0001 C CNN
@@
 Wire Wire Line
 	6100 3850 6000 3850
-$Comp
-L GND #PWR010
-U 1 1 5AD6A0D0
-P 6000 3850
-F 0 "#PWR010" H 6000 3600 50  0001 C CNN
-F 1 "GND" H 6000 3700 50  0000 C CNN
-F 2 "" H 6000 3850 50  0001 C CNN
-F 3 "" H 6000 3850 50  0001 C CNN
-	1    6000 3850
-	0    1    1    0
-$EndComp
 Text GLabel 9650 3600 2    60   Input ~ 0
 IO23
@@
 P1
 Text GLabel 7800 4850 0    60   Input ~ 0
-P3
+P2
 Text GLabel 9100 5400 3    60   Input ~ 0
 P3
@@
 F 0 "J4" H 2100 2750 50  0000 C CNN
 F 1 "Serial" H 2100 2450 50  0000 C CNN
-F 2 "" H 2100 2650 50  0001 C CNN
+F 2 "Wire_Pads:SolderWirePad_2x_1mmDrill" H 2100 2650 50  0001 C CNN
 F 3 "" H 2100 2650 50  0001 C CNN
 	1    2100 2650
@@
 Text GLabel 2300 2650 2    60   Input ~ 0
 RX
-$Comp
-L Conn_01x04 J5
-U 1 1 5AD6B686
-P 2100 3250
-F 0 "J5" H 2100 3450 50  0000 C CNN
-F 1 "Pennies" H 2100 2950 50  0000 C CNN
-F 2 "" H 2100 3250 50  0001 C CNN
-F 3 "" H 2100 3250 50  0001 C CNN
-	1    2100 3250
-	-1   0    0    1
-$EndComp
-Text GLabel 2300 3350 2    60   Input ~ 0
-P0
-Text GLabel 2300 3250 2    60   Input ~ 0
-P1
-Text GLabel 2300 3150 2    60   Input ~ 0
-P2
-Text GLabel 2300 3050 2    60   Input ~ 0
-P3
 Text GLabel 1350 2950 2    60   Input ~ 0
 IO34
@@
 F 0 "J1" H 1150 3350 50  0000 C CNN
 F 1 "Left2" H 1150 2850 50  0000 C CNN
-F 2 "" H 1150 3150 50  0001 C CNN
+F 2 "Wire_Pads:SolderWirePad_4xInline_1mmDrill" H 1150 3150 50  0001 C CNN
 F 3 "" H 1150 3150 50  0001 C CNN
 	1    1150 3150
@@
 F 0 "J2" H 1150 3750 50  0000 C CNN
 F 1 "Left3" H 1150 3450 50  0000 C CNN
-F 2 "" H 1150 3650 50  0001 C CNN
+F 2 "Wire_Pads:SolderWirePad_2x_1mmDrill" H 1150 3650 50  0001 C CNN
 F 3 "" H 1150 3650 50  0001 C CNN
 	1    1150 3650
@@
 L Conn_01x09 J3
 U 1 1 5AD7D502
-P 2100 4050
-F 0 "J3" H 2100 4550 50  0000 C CNN
-F 1 "Bottom" H 2100 3550 50  0000 C CNN
-F 2 "" H 2100 4050 50  0001 C CNN
-F 3 "" H 2100 4050 50  0001 C CNN
-	1    2100 4050
-	-1   0    0    1
-$EndComp
-Text GLabel 2300 3650 2    60   Input ~ 0
+P 2050 3400
+F 0 "J3" H 2050 3900 50  0000 C CNN
+F 1 "Bottom" H 2050 2900 50  0000 C CNN
+F 2 "" H 2050 3400 50  0001 C CNN
+F 3 "" H 2050 3400 50  0001 C CNN
+	1    2050 3400
+	-1   0    0    1
+$EndComp
+Text GLabel 2250 3000 2    60   Input ~ 0
 IO13
-Text GLabel 2300 3750 2    60   Input ~ 0
+Text GLabel 2250 3100 2    60   Input ~ 0
 SD2
-Text GLabel 2300 3850 2    60   Input ~ 0
+Text GLabel 2250 3200 2    60   Input ~ 0
 SD3
-Text GLabel 2300 3950 2    60   Input ~ 0
+Text GLabel 2250 3300 2    60   Input ~ 0
 CMD
-Text GLabel 2300 4050 2    60   Input ~ 0
+Text GLabel 2250 3400 2    60   Input ~ 0
 CLK
-Text GLabel 2300 4150 2    60   Input ~ 0
+Text GLabel 2250 3500 2    60   Input ~ 0
 SD0
-Text GLabel 2300 4250 2    60   Input ~ 0
+Text GLabel 2250 3600 2    60   Input ~ 0
 SD1
-NoConn ~ 2300 4350
-Text GLabel 2300 4450 2    60   Input ~ 0
+NoConn ~ 2250 3700
+Text GLabel 2250 3800 2    60   Input ~ 0
 IO2
 $Comp
@@
 F 0 "J6" H 2900 2750 50  0000 C CNN
 F 1 "Right1" H 2900 2450 50  0000 C CNN
-F 2 "" H 2900 2650 50  0001 C CNN
+F 2 "Wire_Pads:SolderWirePad_2x_1mmDrill" H 2900 2650 50  0001 C CNN
 F 3 "" H 2900 2650 50  0001 C CNN
 	1    2900 2650
@@
 F 0 "J7" H 2900 3050 50  0000 C CNN
 F 1 "Right2" H 2900 2850 50  0000 C CNN
-F 2 "" H 2900 2950 50  0001 C CNN
+F 2 "Wire_Pads:SolderWirePad_single_1mmDrill" H 2900 2950 50  0001 C CNN
 F 3 "" H 2900 2950 50  0001 C CNN
 	1    2900 2950
@@
 F 0 "J9" H 2900 4100 50  0000 C CNN
 F 1 "Right4" H 2900 3900 50  0000 C CNN
-F 2 "" H 2900 4000 50  0001 C CNN
+F 2 "Wire_Pads:SolderWirePad_single_1mmDrill" H 2900 4000 50  0001 C CNN
 F 3 "" H 2900 4000 50  0001 C CNN
 	1    2900 4000
@@
 IO0
 $Comp
-L VSS #PWR011
+L VSS #PWR07
 U 1 1 5AD7EECF
 P 1750 6400
-F 0 "#PWR011" H 1750 6250 50  0001 C CNN
+F 0 "#PWR07" H 1750 6250 50  0001 C CNN
 F 1 "VSS" H 1750 6550 50  0000 C CNN
 F 2 "" H 1750 6400 50  0001 C CNN
@@
 $EndComp
 $Comp
-L VDD #PWR012
+L VDD #PWR08
 U 1 1 5AD7EF29
 P 1750 6100
-F 0 "#PWR012" H 1750 5950 50  0001 C CNN
+F 0 "#PWR08" H 1750 5950 50  0001 C CNN
 F 1 "VDD" H 1750 6250 50  0000 C CNN
 F 2 "" H 1750 6100 50  0001 C CNN
@@
 F 0 "J10" H 1150 2750 50  0000 C CNN
 F 1 "Left1" H 1150 2450 50  0000 C CNN
-F 2 "" H 1150 2650 50  0001 C CNN
+F 2 "Connectors:GS2" H 1150 2650 50  0001 C CNN
 F 3 "" H 1150 2650 50  0001 C CNN
 	1    1150 2650
@@
 Connection ~ 4850 1400
 Connection ~ 1750 6400
+$Comp
+L Conn_01x01 J13
+U 1 1 5AF8C2A5
+P 1200 4950
+F 0 "J13" H 1200 5050 50  0000 C CNN
+F 1 "Penny0" H 1200 4850 50  0000 C CNN
+F 2 "Wire_Pads:Penny" H 1200 4950 50  0001 C CNN
+F 3 "" H 1200 4950 50  0001 C CNN
+	1    1200 4950
+	-1   0    0    1
+$EndComp
+$Comp
+L Conn_01x01 J12
+U 1 1 5AF8C41B
+P 1200 4650
+F 0 "J12" H 1200 4750 50  0000 C CNN
+F 1 "Penny1" H 1200 4550 50  0000 C CNN
+F 2 "Wire_Pads:Penny" H 1200 4650 50  0001 C CNN
+F 3 "" H 1200 4650 50  0001 C CNN
+	1    1200 4650
+	-1   0    0    1
+$EndComp
+$Comp
+L Conn_01x01 J5
+U 1 1 5AF8C77A
+P 1200 4050
+F 0 "J5" H 1200 4150 50  0000 C CNN
+F 1 "Penny3" H 1200 3950 50  0000 C CNN
+F 2 "Wire_Pads:Penny" H 1200 4050 50  0001 C CNN
+F 3 "" H 1200 4050 50  0001 C CNN
+	1    1200 4050
+	-1   0    0    1
+$EndComp
+$Comp
+L Conn_01x01 J11
+U 1 1 5AF8C780
+P 1200 4350
+F 0 "J11" H 1200 4450 50  0000 C CNN
+F 1 "Penny2" H 1200 4250 50  0000 C CNN
+F 2 "Wire_Pads:Penny" H 1200 4350 50  0001 C CNN
+F 3 "" H 1200 4350 50  0001 C CNN
+	1    1200 4350
+	-1   0    0    1
+$EndComp
+Text GLabel 1400 4050 2    60   Input ~ 0
+P3
+Text GLabel 1400 4350 2    60   Input ~ 0
+P2
+Text GLabel 1400 4950 2    60   Input ~ 0
+P0
+Text GLabel 1400 4650 2    60   Input ~ 0
+P1
+$Comp
+L VSS #PWR09
+U 1 1 5AF92473
+P 6000 3850
+F 0 "#PWR09" H 6000 3700 50  0001 C CNN
+F 1 "VSS" H 6000 4000 50  0000 C CNN
+F 2 "" H 6000 3850 50  0001 C CNN
+F 3 "" H 6000 3850 50  0001 C CNN
+	1    6000 3850
+	1    0    0    -1
+$EndComp
+$Comp
+L VSS #PWR010
+U 1 1 5AF924FD
+P 9900 5000
+F 0 "#PWR010" H 9900 4850 50  0001 C CNN
+F 1 "VSS" H 9900 5150 50  0000 C CNN
+F 2 "" H 9900 5000 50  0001 C CNN
+F 3 "" H 9900 5000 50  0001 C CNN
+	1    9900 5000
+	0    1    1    0
+$EndComp
+$Comp
+L VSS #PWR011
+U 1 1 5AF92587
+P 7650 5050
+F 0 "#PWR011" H 7650 4900 50  0001 C CNN
+F 1 "VSS" H 7650 5200 50  0000 C CNN
+F 2 "" H 7650 5050 50  0001 C CNN
+F 3 "" H 7650 5050 50  0001 C CNN
+	1    7650 5050
+	0    -1   -1   0
+$EndComp
+$Comp
+L VSS #PWR012
+U 1 1 5AF92611
+P 8300 5500
+F 0 "#PWR012" H 8300 5350 50  0001 C CNN
+F 1 "VSS" H 8300 5650 50  0000 C CNN
+F 2 "" H 8300 5500 50  0001 C CNN
+F 3 "" H 8300 5500 50  0001 C CNN
+	1    8300 5500
+	-1   0    0    1
+$EndComp
+$Comp
+L Conn_01x02 J14
+U 1 1 5AF927B2
+P 2350 4700
+F 0 "J14" H 2350 4800 50  0000 C CNN
+F 1 "Power" H 2350 4500 50  0000 C CNN
+F 2 "Wire_Pads:SolderWirePad_2x_1mmDrill" H 2350 4700 50  0001 C CNN
+F 3 "" H 2350 4700 50  0001 C CNN
+	1    2350 4700
+	-1   0    0    1
+$EndComp
+$Comp
+L VSS #PWR013
+U 1 1 5AF92923
+P 2550 4600
+F 0 "#PWR013" H 2550 4450 50  0001 C CNN
+F 1 "VSS" H 2550 4750 50  0000 C CNN
+F 2 "" H 2550 4600 50  0001 C CNN
+F 3 "" H 2550 4600 50  0001 C CNN
+	1    2550 4600
+	0    1    1    0
+$EndComp
+$Comp
+L VDD #PWR014
+U 1 1 5AF92987
+P 2550 4700
+F 0 "#PWR014" H 2550 4550 50  0001 C CNN
+F 1 "VDD" H 2550 4850 50  0000 C CNN
+F 2 "" H 2550 4700 50  0001 C CNN
+F 3 "" H 2550 4700 50  0001 C CNN
+	1    2550 4700
+	0    1    1    0
+$EndComp
+$Comp
+L Conn_01x02 J15
+U 1 1 5AF92DFF
+P 3200 4600
+F 0 "J15" H 3200 4700 50  0000 C CNN
+F 1 "Right5" H 3200 4400 50  0000 C CNN
+F 2 "Connectors:GS2" H 3200 4600 50  0001 C CNN
+F 3 "" H 3200 4600 50  0001 C CNN
+	1    3200 4600
+	-1   0    0    1
+$EndComp
+Text GLabel 3400 4500 2    60   Input ~ 0
+IO16
+Text GLabel 3400 4600 2    60   Input ~ 0
+IO17
 $EndSCHEMATC
