File: schematic/_saved_badge.sch (KiCad schematic (older format))
At the start: 42 parts, among them J1 Left2, J10 Left1, J11 Penny2, J12 Penny1, J13 Penny0, J14 Power, J15 Right5, J2 Left3, J3 Bottom, J4 Serial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

Commit message: New board revision
Connections:
- net GND: no longer LS1.1
- net IO13: now also LS1.1
Changed lines of the file:
@@
 $EndComp
 Text GLabel 5650 5000 1    60   Input ~ 0
-IO2
+IO13
 $Comp
 L VSS #PWR015
@@
 $EndComp
 $Comp
-L GND #PWR?
+L GND #PWR016
 U 1 1 5B16A9F1
 P 2700 5450
-F 0 "#PWR?" H 2700 5200 50  0001 C CNN
+F 0 "#PWR016" H 2700 5200 50  0001 C CNN
 F 1 "GND" H 2700 5300 50  0000 C CNN
 F 2 "" H 2700 5450 50  0001 C CNN
