File: schematic/_autosave-badge.kicad_pcb (KiCad board)
At the start: 2 copper layers, 90.2 x 45.7 mm, 50 parts, among them J1 Left2, J10 Left1, J11 Penny2, J12 Penny1, J13 Penny0, J14 Power, J15 Right5, J2 Left3, J4 Serial, J5 Penny3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

Commit message: Checking for update
Parts:
- removed LED1, LED10, LED2, LED3, LED4, LED5, LED6, LED7, LED8, LED9: WS2812B, LEDs:LED_WS2812B-PLCC4
