File: schematic/badge.sch (KiCad schematic (older format))
At the start: 36 parts, among them J1 Left2, J10 Left1, J2 Left3, J3 Bottom, J4 Serial, J5 Pennies, J6 Right1, J7 Right2, J8 Right3, J9 Right4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

Commit message: Checking for update
Parts:
- removed J5: Pennies, symbol Conn_01x04
- added J11: Penny2, Wire_Pads:Penny, symbol Conn_01x01
- added J12: Penny1, Wire_Pads:Penny, symbol Conn_01x01
- added J13: Penny0, Wire_Pads:Penny, symbol Conn_01x01
- added J14: Power, Wire_Pads:SolderWirePad_2x_1mmDrill, symbol Conn_01x02
- added J15: Right5, Connectors:GS2, symbol Conn_01x02
- added J5: Penny3, Wire_Pads:Penny, symbol Conn_01x01
- added LS1: PKMCS0909E4000-R1, PKMCS0909E4000-R1:XDCR_PKMCS0909E4000-R1, symbol PKMCS0909E4000-R1
- J1: footprint (none) -> Wire_Pads:SolderWirePad_4xInline_1mmDrill
- J10: footprint (none) -> Connectors:GS2
- J2, J4, J6: footprint (none) -> Wire_Pads:SolderWirePad_2x_1mmDrill
- J7, J9: footprint (none) -> Wire_Pads:SolderWirePad_single_1mmDrill
Connections:
- net GND: no longer C11.2, U1.1 (GND), U1.15 (GND), U1.38 (GND), U1.39 (GND-PAD)
- net IO16: now also J15.2 (Pin_2)
- net IO17: now also J15.1 (Pin_1)
- net IO2: now also LS1.1
- net P0: now also J13.1 (Pin_1)
- net P1: now also J12.1 (Pin_1)
- net P2: now also U1.13 (IO14), J11.1 (Pin_1)
- net P3: now also J5.1 (Pin_1); no longer U1.13 (IO14)
- net VDD: now also J14.1 (Pin_1)
- net VSS: now also C11.2, U1.1 (GND), U1.15 (GND), U1.38 (GND), U1.39 (GND-PAD), J14.2 (Pin_2), LS1.2
Other:
- moved on the sheet: J3
