File: Schematic/V2/_autosave-badge.kicad_pcb (KiCad board)
At the start: 2 copper layers, 90.2 x 45.7 mm, 52 parts, among them J1 Left2, J10 USB_B_Micro, J11 Penny2, J12 Penny1, J13 Penny0, J14 Power, J15 Right5, J4 Serial, J5 Penny3, J6 Right1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

Commit message: Added charging hardware
Parts:
- removed C14, C17: 4.7uF, Capacitors_SMD:C_0805_HandSoldering
- removed C15, C19: 0.1uF, Capacitors_SMD:C_0805_HandSoldering
- removed C16, C18: 1uF, Capacitors_SMD:C_0805_HandSoldering
- removed J8: Right3, Pin_Headers:Pin_Header_Straight_1x05_Pitch2.54mm
- removed R2: 2k, Resistors_SMD:R_0805_HandSoldering
- removed U2: otter_CH330, Housings_SOIC:SOIC-8-1EP_3.9x4.9mm_Pitch1.27mm
- removed U4: TLV1117-33, TO_SOT_Packages_SMD:SOT-223-3_TabPin2
- added J2: Left3, Wire_Pads:SolderWirePad_2x_1mmDrill, F.Cu at (148.2, 106.4)
- 0001, 0010, 0100, 0101, 0110, 1000, 1001, 1010, 1100, 1110: footprint Badge:WS2812B-Sunken -> LEDs:LED_WS2812B-PLCC4; moved to B.Cu
- C1, C10, C2, C3, C4, C5, C6, C7, C8, C9: moved to B.Cu
- J10: value USB_B_Micro -> Left1; footprint Connectors_USB:USB_Micro-B_Molex_47346-0001 -> Connectors:GS2
- moved G*** 113.9 mm to (126.5, 64.4)
- moved ? 108.5 mm to (145.8, 85.7)
- moved J10 75.9 mm to (158.3, 106.4), turned to 90 degrees
- moved J1 54.2 mm to (147.6, 102.2)
- moved 0001 40.3 mm to (103.7, 108.0)
- moved 0010 40.3 mm to (139.2, 108.0)
- moved 0100 40.3 mm to (157.0, 108.0)
- moved 0110 40.3 mm to (121.4, 108.0)
- moved 1001 40.3 mm to (94.8, 108.0)
- moved 1010 40.3 mm to (130.3, 108.0)
- moved 1100 40.3 mm to (148.1, 108.0)
- moved 1110 40.3 mm to (112.6, 108.0)
- moved 0101 40.3 mm to (86.4, 107.9)
- moved C10 40.3 mm to (84.4, 111.8)
- moved 1000 40.3 mm to (165.6, 107.9)
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Connections:
- net Net-(U1-Pad11) renamed IO26
- net Net-(U1-Pad17) renamed SD2
- net Net-(U1-Pad18) renamed SD3
- net Net-(U1-Pad19) renamed CMD
- net Net-(U1-Pad20) renamed CLK
- net Net-(U1-Pad21) renamed SD0
- net Net-(U1-Pad22) renamed SD1
- BT1 pad 1: VDDA -> VDD
- J1 pad 1: IO33 -> IO34
- J10 pad 1: VBUS -> VN
- J10 pad 2: Net-(J10-Pad2) -> VP
- J4 pad 1: RX -> TX
- U1 pad 4: Net-(U1-Pad4) -> VP
- U1 pad 5: Net-(U1-Pad5) -> VN
Routing:
- net VSS: track 7.06 -> 88.8 mm, vias 4 -> 14
- net VDD: track 77.6 -> 8.94 mm, vias 19 -> 3
- net SPI: track 0.00 -> 32.0 mm, vias 0 -> 1
- net IO33: track 0.00 -> 25.2 mm, vias 0 -> 2
- net IO32: track 0.00 -> 14.7 mm
- net IO35: track 0.00 -> 12.1 mm
- net IO34: track 0.00 -> 10.4 mm
- net IO27: track 0.00 -> 5.03 mm
- net P3: track 66.4 -> 70.6 mm
- net IO26: track 0.00 -> 4.05 mm
- net VP: track 0.00 -> 3.95 mm
- net VN: track 0.00 -> 3.94 mm
- net P2: track 51.2 -> 53.5 mm
- net Net-(LED10-Pad4): track 4.63 -> 5.22 mm
