File: Schematic/V2/badge.sch (KiCad schematic (older format))
At the start: 50 parts, among them J1 Left2, J10 USB_B_Micro, J11 Penny2, J12 Penny1, J13 Penny0, J14 Power, J15 Right5, J4 Serial, J5 Penny3, J6 Right1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

Commit message: Added charging hardware
Parts:
- removed C14, C17: 4.7uF, Capacitors_SMD:C_0805_HandSoldering, symbol badge-rescue:C
- removed C15, C19: 0.1uF, Capacitors_SMD:C_0805_HandSoldering, symbol badge-rescue:C
- removed C16, C18: 1uF, Capacitors_SMD:C_0805_HandSoldering, symbol badge-rescue:C
- removed J10: USB_B_Micro, Connectors_USB:USB_Micro-B_Molex_47346-0001, symbol Connector:USB_B_Micro
- removed R2: 2k, Resistors_SMD:R_0805_HandSoldering, symbol badge-rescue:R
- removed U2: otter_CH330, Housings_SOIC:SOIC-8-1EP_3.9x4.9mm_Pitch1.27mm, symbol CH330-cache:otter_CH330
- removed U3: MCP73831-2-OT, Package_TO_SOT_SMD:SOT-23-5, symbol Battery_Management:MCP73831-2-OT
- removed U4: TLV1117-33, TO_SOT_Packages_SMD:SOT-223-3_TabPin2, symbol Regulator_Linear:TLV1117-33
- added J2: Left3, Wire_Pads:SolderWirePad_2x_1mmDrill, symbol badge-rescue:Conn_01x02
- added J3: Bottom, symbol badge-rescue:Conn_01x09
Connections:
- net labels added: CLK, CMD, IO2, IO26, SD0, SD1, SD2, SD3, VN, VP
- net labels removed: VBUS, VDDA
- wire segments 133 -> 113
- no-connect marks 12 -> 3
Other:
- note removed: "Check if is 3v output later\n"
- moved on the sheet: BT1, J11, J12, J13, J14, J15, J5, LS1
