File: Schematic/badge.kicad_pcb (KiCad board)
At the start: 2 copper layers, 90.2 x 45.7 mm, 42 parts, among them J1 Left2, J10 Left1, J11 Penny2, J12 Penny1, J13 Penny0, J14 Power, J15 Right5, J2 Left3, J4 Serial, J5 Penny3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

Commit message: Added charging hardware
Parts:
- removed J2: Left3, Wire_Pads:SolderWirePad_2x_1mmDrill
- added C14: 4.7uF, Capacitors_SMD:C_0805_HandSoldering, F.Cu at (89.1, 119.9)
- added C15: 0.1uF, Capacitors_SMD:C_0805_HandSoldering, F.Cu at (97.8, 115.1)
- added C16: 1uF, Capacitors_SMD:C_0805_HandSoldering, F.Cu at (106.1, 119.9)
- added C17: 4.7uF, Capacitors_SMD:C_0805_HandSoldering, F.Cu at (98.1, 111.4)
- added C18: 1uF, Capacitors_SMD:C_0805_HandSoldering, F.Cu at (101.1, 119.9)
- added C19: 0.1uF, Capacitors_SMD:C_0805_HandSoldering, F.Cu at (94.1, 119.9)
- added G***: LOGO, Badge:Bsides, F.Cu at (13.2, 76.6)
- added J8: Right3, Pin_Headers:Pin_Header_Straight_1x05_Pitch2.54mm, F.Cu at (122.0, 130.1)
- added R2: 2k, Resistors_SMD:R_0805_HandSoldering, F.Cu at (98.1, 108.4)
- added R3: 0ohm, Resistors_SMD:R_0805_HandSoldering, F.Cu at (110.7, 113.2)
- added R4: 22ohm, Resistors_SMD:R_0805_HandSoldering, F.Cu at (135.9, 123.0)
- added U2: otter_CH330, Housings_SOIC:SOIC-8_3.9x4.9mm_Pitch1.27mm, F.Cu at (92.5, 115.6)
- added U3: MCP73831-2-OT, TO_SOT_Packages_SMD:SOT-23-5_HandSoldering, F.Cu at (91.8, 110.6)
- added U4: TLV1117-33, TO_SOT_Packages_SMD:SOT-223-3_TabPin2, F.Cu at (105.3, 113.5)
- 0001, 0010, 0100, 0101, 0110, 1000, 1001, 1010, 1100, 1110: footprint LEDs:LED_WS2812B-PLCC4 -> Badge:WS2812B-Sunken; moved to F.Cu
- C1, C10, C11, C12, C13, C2, C3, C4, C5, C6, C7, C8, C9, R1: moved to F.Cu
- J10: value Left1 -> USB_B_Micro; footprint Connectors:GS2 -> Connectors_USB:USB_Micro-B_Molex_47346-0001
- LS1: value Piezo -> PKMCS0909E4000-R1
- moved ? 87.9 mm to (38.1, 98.9)
- moved J10 75.9 mm to (82.8, 114.3), turned to 270 degrees
- moved J1 54.2 mm to (201.7, 97.9)
- moved C11 14.4 mm to (162.3, 106.6), turned to 0 degrees
- moved C4 12.6 mm to (138.9, 99.3)
- moved C6 12.6 mm to (121.3, 99.3)
- moved C2 12.6 mm to (156.9, 99.3)
- moved 0010 12.6 mm to (140.4, 95.4)
- moved 0100 12.6 mm to (158.2, 95.4)
- moved 0001 12.6 mm to (104.9, 95.4)
- moved 0110 12.6 mm to (122.6, 95.4)
- moved 1001 12.6 mm to (96.0, 95.4)
- moved 1010 12.6 mm to (131.5, 95.4)
- moved 1100 12.6 mm to (149.3, 95.4)
- moved 1110 12.6 mm to (113.8, 95.4)
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Connections:
- net CLK renamed Net-(U1-Pad20)
- net CMD renamed Net-(U1-Pad19)
- net IO26 renamed Net-(U1-Pad11)
- net SD0 renamed Net-(U1-Pad21)
- net SD1 renamed Net-(U1-Pad22)
- net SD2 renamed Net-(U1-Pad17)
- net SD3 renamed Net-(U1-Pad18)
- BT1 pad 1: VDD -> VDDA
- C12 pad 1: VSS -> GND
- C13 pad 1: VSS -> GND
- J1 pad 1: IO34 -> IO33
- J10 pad 1: VN -> VBUS
- J10 pad 2: VP -> Net-(J10-Pad2)
- J14 pad 1: VSS -> VDD
- J4 pad 1: TX -> RX
- LS1 pad 1: IO13 -> Net-(LS1-Pad1)
- U1 pad 13: P2 -> P3
- U1 pad 14: P1 -> P2
- U1 pad 23: P3 -> P1
- U1 pad 4: VP -> Net-(U1-Pad4)
- U1 pad 5: VN -> Net-(U1-Pad5)
Routing:
- net VSS: track 92.7 -> 5.17 mm, vias 15 -> 3
- net VDD: track 6.40 -> 88.1 mm, vias 1 -> 20
- net P3: track 77.7 -> 1.27 mm
- net TX: track 13.5 -> 82.8 mm, vias 0 -> 2
- net RX: track 10.7 -> 79.3 mm, vias 0 -> 2
- net P2: track 52.7 -> 7.62 mm
- net VDDA: track 0.00 -> 32.9 mm
- net SPI: track 32.0 -> 0.00 mm, vias 1 -> 0
- net VBUS: track 0.00 -> 25.4 mm
- net IO33: track 25.2 -> 0.00 mm, vias 2 -> 0
- net IO32: track 14.7 -> 0.00 mm
- net IO35: track 12.1 -> 0.00 mm
- net Net-(LS1-Pad1): track 0.00 -> 10.7 mm, vias 0 -> 1
- net IO34: track 10.4 -> 0.00 mm
- net Net-(R2-Pad1): track 0.00 -> 8.62 mm
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Other:
- board text added: "Expansion Port"
- board text added: "v3"
- board text removed: "Proposed BSides Iowa 2018 Badge!"
- board text removed: "WR"
- board text removed: "v2"

Commit message: Added charging hardware
Routing:
- net VDDA: track 32.9 -> 37.5 mm
- net VDD: vias 20 -> 22
Changed lines of the file:
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@@
     (thickness 1.6)
     (drawings 20)
-    (tracks 257)
+    (tracks 261)
     (zones 0)
     (modules 55)
@@
   (gr_line (start 171.45 96.52) (end 171.45 142.24) (angle 90) (layer Eco1.User) (width 0.2))
   (gr_line (start 81.28 96.52) (end 171.45 96.52) (angle 90) (layer Eco1.User) (width 0.2))
+  (via (at 104.12 110.397) (size 0.6) (drill 0.4) (layers F.Cu B.Cu) (net 1))
+  (via (at 106.32 110.397) (size 0.6) (drill 0.4) (layers F.Cu B.Cu) (net 1))
   (segment (start 84.62 93.828576) (end 84.92 93.828576) (width 0.25) (layer F.Cu) (net 1))
   (segment (start 83.77 94.678576) (end 84.62 93.828576) (width 0.25) (layer F.Cu) (net 1))
@@
   (segment (start 104.945 119.897) (end 107.62 117.222) (width 0.25) (layer F.Cu) (net 38))
   (segment (start 104.82 119.897) (end 104.945 119.897) (width 0.25) (layer F.Cu) (net 38))
+  (segment (start 110.744 114.273) (end 110.744 114.507) (width 0.25) (layer F.Cu) (net 38))
+  (segment (start 113.87 111.147) (end 110.744 114.273) (width 0.25) (layer F.Cu) (net 38))
   (segment (start 89.969 109.601) (end 90.424 109.601) (width 0.25) (layer F.Cu) (net 39))
   (segment (start 89.394 110.176) (end 89.969 109.601) (width 0.25) (layer F.Cu) (net 39))
@@
     (connect_pads (clearance 0.508))
     (min_thickness 0.254)
-    (fill (arc_segments 16) (thermal_gap 0.508) (thermal_bridge_width 0.508))
+    (fill yes (arc_segments 16) (thermal_gap 0.508) (thermal_bridge_width 0.508))
     (polygon
       (pts
@@
     (connect_pads (clearance 0.508))
     (min_thickness 0.254)
-    (fill (arc_segments 16) (thermal_gap 0.508) (thermal_bridge_width 0.508))
+    (fill yes (arc_segments 16) (thermal_gap 0.508) (thermal_bridge_width 0.508))
     (polygon
       (pts

Commit message: Added charging hardware
Routing:
- net P3: track 1.27 -> 69.1 mm
- net IO27: track 0.00 -> 59.6 mm, vias 0 -> 2
- net P2: track 7.62 -> 60.7 mm
- net VSS: track 5.17 -> 12.9 mm, vias 3 -> 5
Changed lines of the file:
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@@
     (thickness 1.6)
     (drawings 20)
-    (tracks 261)
+    (tracks 293)
     (zones 0)
     (modules 55)
@@
   (gr_line (start 171.45 96.52) (end 171.45 142.24) (angle 90) (layer Eco1.User) (width 0.2))
   (gr_line (start 81.28 96.52) (end 171.45 96.52) (angle 90) (layer Eco1.User) (width 0.2))
+  (via (at 96.92 111.197) (size 0.6) (drill 0.4) (layers F.Cu B.Cu) (net 2))
+  (via (at 99.12 108.397) (size 0.6) (drill 0.4) (layers F.Cu B.Cu) (net 2))
   (via (at 104.12 110.397) (size 0.6) (drill 0.4) (layers F.Cu B.Cu) (net 1))
   (via (at 106.32 110.397) (size 0.6) (drill 0.4) (layers F.Cu B.Cu) (net 1))
@@
   (via (at 162.814 125.984) (size 0.6) (drill 0.4) (layers F.Cu B.Cu) (net 2))
   (segment (start 144.43028 125.39472) (end 144.73 125.095) (width 0.25) (layer F.Cu) (net 2))
+  (segment (start 96.92 110.597) (end 99.12 108.397) (width 0.25) (layer B.Cu) (net 2))
+  (segment (start 96.92 111.197) (end 96.92 110.597) (width 0.25) (layer B.Cu) (net 2))
+  (segment (start 95.974 110.551) (end 96.82 111.397) (width 0.25) (layer F.Cu) (net 2))
+  (segment (start 93.124 110.551) (end 95.974 110.551) (width 0.25) (layer F.Cu) (net 2))
   (segment (start 164.145 96.865576) (end 164.145 97.003576) (width 0.25) (layer F.Cu) (net 4))
   (segment (start 161.105 93.825576) (end 164.145 96.865576) (width 0.25) (layer F.Cu) (net 4))
@@
   (segment (start 146.22 130.64) (end 146.22 128.38) (width 0.25) (layer F.Cu) (net 26))
   (segment (start 93.98 142.24) (end 93.98 140.97) (width 0.25) (layer F.Cu) (net 27))
+  (segment (start 112.07301 124.14699) (end 94.38001 141.83999) (width 0.25) (layer F.Cu) (net 27))
+  (segment (start 128.971012 124.14699) (end 112.07301 124.14699) (width 0.25) (layer F.Cu) (net 27))
+  (segment (start 144.313012 108.80499) (end 128.971012 124.14699) (width 0.25) (layer F.Cu) (net 27))
+  (segment (start 146.541019 108.80499) (end 144.313012 108.80499) (width 0.25) (layer F.Cu) (net 27))
+  (segment (start 147.49 109.753971) (end 146.541019 108.80499) (width 0.25) (layer F.Cu) (net 27))
+  (segment (start 147.49 110.38) (end 147.49 109.753971) (width 0.25) (layer F.Cu) (net 27))
   (segment (start 137.22 122.997) (end 137.22 119.497) (width 0.25) (layer F.Cu) (net 28))
   (segment (start 141.782 114.935) (end 144.73 114.935) (width 0.25) (layer F.Cu) (net 28))
@@
   (segment (start 137.16 126.182) (end 139.517 123.825) (width 0.25) (layer F.Cu) (net 29))
   (segment (start 137.16 142.24) (end 137.16 126.182) (width 0.25) (layer F.Cu) (net 29))
+  (via (at 94.52 111.597) (size 0.6) (drill 0.4) (layers F.Cu B.Cu) (net 30))
+  (segment (start 93.124 111.501) (end 94.424 111.501) (width 0.25) (layer F.Cu) (net 30))
+  (segment (start 94.424 111.501) (end 94.52 111.597) (width 0.25) (layer F.Cu) (net 30))
+  (segment (start 131.805001 112.279999) (end 132.522002 112.997) (width 0.25) (layer B.Cu) (net 30))
+  (segment (start 121.284999 112.279999) (end 131.805001 112.279999) (width 0.25) (layer B.Cu) (net 30))
+  (segment (start 120.567998 112.997) (end 121.284999 112.279999) (width 0.25) (layer B.Cu) (net 30))
+  (segment (start 94.52 111.597) (end 95.92 112.997) (width 0.25) (layer B.Cu) (net 30))
+  (segment (start 95.92 112.997) (end 120.567998 112.997) (width 0.25) (layer B.Cu) (net 30))
+  (via (at 148.92 112.797) (size 0.6) (drill 0.4) (layers F.Cu B.Cu) (net 30))
+  (segment (start 132.522002 112.997) (end 148.72 112.997) (width 0.25) (layer B.Cu) (net 30))
+  (segment (start 148.72 112.997) (end 148.92 112.797) (width 0.25) (layer B.Cu) (net 30))
+  (segment (start 148.92 110.54) (end 148.76 110.38) (width 0.25) (layer F.Cu) (net 30))
+  (segment (start 148.92 112.797) (end 148.92 110.54) (width 0.25) (layer F.Cu) (net 30))
   (segment (start 158.82 106.647) (end 161.07 106.647) (width 0.25) (layer F.Cu) (net 35))
   (segment (start 160.19 108.88) (end 160.19 110.38) (width 0.25) (layer F.Cu) (net 35))
@@
   (segment (start 161.07 106.647) (end 161.07 107.522) (width 0.25) (layer F.Cu) (net 35))
   (segment (start 115.57 142.24) (end 115.57 134.62) (width 0.25) (layer F.Cu) (net 36))
+  (segment (start 145.52 110.38) (end 136.12 119.78) (width 0.25) (layer F.Cu) (net 36))
+  (segment (start 146.22 110.38) (end 145.52 110.38) (width 0.25) (layer F.Cu) (net 36))
+  (segment (start 136.12 119.78) (end 136.12 124.597) (width 0.25) (layer F.Cu) (net 36))
+  (segment (start 136.12 124.597) (end 121.32 124.597) (width 0.25) (layer F.Cu) (net 36))
+  (segment (start 121.32 124.597) (end 116.32 129.597) (width 0.25) (layer F.Cu) (net 36))
+  (segment (start 116.32 141.49) (end 115.97001 141.83999) (width 0.25) (layer F.Cu) (net 36))
+  (segment (start 116.32 129.597) (end 116.32 141.49) (width 0.25) (layer F.Cu) (net 36))
   (segment (start 109.844 114.507) (end 110.744 114.507) (width 0.25) (layer F.Cu) (net 38))
   (segment (start 109.56 114.507) (end 109.844 114.507) (width 0.25) (layer F.Cu) (net 38))

Commit message: Ordered V3
Parts:
- removed ?: 1pin, Connectors:1pin
- removed G***: LOGO, Badge:Bsides
- removed J15: Right5, Connectors:GS2
- removed J6: Right1, Wire_Pads:SolderWirePad_2x_1mmDrill
- added REF**: Binder, Badge:Binder, B.Cu at (126.5, 103.6)
- J1: footprint Wire_Pads:SolderWirePad_4xInline_1mmDrill -> Pin_Headers:Pin_Header_Straight_1x04_Pitch2.54mm
- moved J1 57.9 mm to (144.4, 106.6), turned to 90 degrees
- moved REF*** 15.6 mm to (112.5, 126.8)
- moved J14 4.31 mm to (83.9, 126.7)
Connections:
- C12 pad 1: GND -> VSS
- C13 pad 1: GND -> VSS
- J14 pad 1: VDD -> VSS
- J4 pad 1: RX -> TX
Routing:
- net SPI: track 0.00 -> 34.5 mm, vias 0 -> 2
- net VSS: track 12.9 -> 45.8 mm
- net IO16: track 3.19 -> 30.0 mm, vias 0 -> 2
- net VDDA: track 37.5 -> 62.9 mm
- net IO5: track 0.00 -> 24.9 mm, vias 0 -> 1
- net IO23: track 25.1 -> 0.24 mm
- net IO18: track 0.00 -> 23.4 mm, vias 0 -> 1
- net IO17: track 3.19 -> 26.4 mm, vias 0 -> 1
- net IO19: track 0.00 -> 21.9 mm, vias 0 -> 1
- net IO22: track 19.3 -> 0.00 mm
- net IO33: track 0.00 -> 10.0 mm
- net VDD: track 88.1 -> 97.9 mm, vias 22 -> 28
- net IO32: track 0.00 -> 8.76 mm
- net IO35: track 0.00 -> 7.59 mm
- net IO34: track 0.00 -> 6.73 mm
Other:
- board size 90.2 x 45.7 mm -> 90.2 x 53.4 mm
