File: Schematic/Badge/badge.kicad_pcb (KiCad board)
At the start: 2 copper layers, 90.2 x 53.4 mm, 52 parts, among them J1 Left2, J10 USB_B_Micro, J11 Penny2, J12 Penny1, J13 Penny0, J14 Power, J4 Serial, J5 Penny3, J7 Right2, J8 Right3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

Commit message: Fixed issues with v3, rearranged caps to make assembly eaiser
Parts:
- moved C14 12.8 mm to (92.7, 107.6), turned to 180 degrees
- moved R3 6.56 mm to (110.0, 106.6), turned to 0 degrees
- moved C15 5.15 mm to (96.6, 120.1), turned to 180 degrees
- moved R4 4.45 mm to (140.3, 122.9), turned to 270 degrees
- moved J14 3.81 mm to (86.7, 129.3), turned to 180 degrees
- moved C17 3.78 mm to (98.1, 107.6)
- moved C19 3.01 mm to (91.1, 120.1)
- moved BT1 2.85 mm to (126.6, 114.0), turned to 0 degrees
- moved R2 2.57 mm to (98.7, 110.9)
- moved C16 1.27 mm to (107.3, 120.1)
- moved C18 1.27 mm to (102.3, 120.1)
- moved J10 1.27 mm to (84.1, 114.6)
- moved U2 1.27 mm to (93.7, 115.8)
- moved U3 1.27 mm to (93.0, 110.8)
- moved U4 1.27 mm to (106.6, 113.8)
Routing:
- net VDDA: track 62.9 -> 39.3 mm
- net Net-(LS1-Pad1): track 10.7 -> 16.8 mm
- net Net-(C15-Pad1): track 2.76 -> 7.75 mm
- net IO13: track 12.9 -> 8.96 mm
- net IO27: track 59.6 -> 56.1 mm
- net VSS: track 45.8 -> 42.6 mm, vias 5 -> 3
- net P2: track 60.7 -> 57.9 mm
- net P1: track 24.6 -> 21.8 mm
- net RX: track 79.3 -> 77.5 mm
- net TX: track 82.8 -> 81.3 mm
- net VDD: track 97.9 -> 96.4 mm
- net Net-(R2-Pad1): track 8.62 -> 7.39 mm
- net VBUS: track 25.4 -> 24.3 mm
Other:
- board size 90.2 x 53.4 mm -> 90.2 x 64.4 mm
- board text added: "Charger Bypass"

Commit message: v4, changes to add all of the best chineseium bits I can find
Parts:
- C14, C17: value 4.7uF -> 10uF
- J10: footprint Connectors_USB:USB_Micro-B_Molex_47346-0001 -> Connectors_USB:USB_Micro-B_Jing
- R2: value 2k -> 1k
- U3: value MCP73831-2-OT -> HX4056; footprint TO_SOT_Packages_SMD:SOT-23-5_HandSoldering -> Badge:HX4056
- moved R2 7.24 mm to (94.5, 105.0)
- moved C14 4.38 mm to (89.2, 105.0), turned to 0 degrees
- moved C17 3.21 mm to (99.9, 105.0), turned to 180 degrees
- moved REF*** 1.80 mm to (110.7, 126.8)
- moved U3 1.50 mm to (93.7, 109.4), turned to 0 degrees
- moved J10 0.91 mm to (83.9, 113.7)
Connections:
- net IO22 renamed Net-(U1-Pad36)
- net IO23 renamed Net-(U1-Pad37)
- J4 pad 1: TX -> RX
- U1 pad 34: RX -> TX
- U1 pad 35: TX -> RX
- U3 pad 1: IO27 -> (no net)
- U3 pad 2: VSS -> Net-(R2-Pad1)
- U3 pad 3: VDDA -> VSS
- U3 pad 5: Net-(R2-Pad1) -> VDDA
Routing:
- net VSS: track 42.6 -> 49.5 mm
- net TX: track 81.3 -> 76.7 mm
- net RX: track 77.5 -> 81.3 mm
- net Net-(R2-Pad1): track 7.39 -> 4.93 mm
- net VBUS: track 24.3 -> 26.5 mm
- net Net-(J10-Pad3): track 4.56 -> 5.95 mm, vias 0 -> 2
- net Net-(LS1-Pad1): track 16.8 -> 15.5 mm
- net VDDA: track 39.3 -> 40.6 mm
- net Net-(J10-Pad2): track 4.82 -> 5.94 mm, vias 2 -> 0
- net IO27: track 56.1 -> 55.1 mm
Other:
- board text added: "v4"
- board text removed: "v3"

Commit message: v5 arrived
Parts:
- added R5: 1.5, Resistors_SMD:R_0805, F.Cu at (83.9, 104.9)
- added Ref**: Val**, NFCBuisness:W, F.Cu at (167.1, 103.6)
- BT1: footprint Battery_Holders:Keystone_3009_1x2450-CoinCell -> Battery_Holders:Keystone_3008_1x2450-CoinCell
- moved J9 60.6 mm to (84.8, 125.1)
- moved R4 19.6 mm to (141.2, 103.4), turned to 180 degrees
- moved C10 4.35 mm to (89.4, 99.3), turned to 180 degrees
- moved U4 3.87 mm to (102.7, 114.1)
- moved C8 3.54 mm to (106.6, 99.3), turned to 180 degrees
- moved C3 3.43 mm to (151.2, 99.3), turned to 180 degrees
- moved C7 3.39 mm to (115.6, 99.3), turned to 180 degrees
- moved C9 3.37 mm to (97.8, 99.3), turned to 180 degrees
- moved C4 3.30 mm to (142.2, 99.3), turned to 180 degrees
- moved C5 3.21 mm to (133.2, 99.3), turned to 180 degrees
- moved C2 3.09 mm to (160.0, 99.3), turned to 180 degrees
- moved C1 3.09 mm to (168.4, 99.2), turned to 180 degrees
- moved C6 3.05 mm to (124.4, 99.3), turned to 180 degrees
- moved BT1 1.70 mm to (125.4, 115.2), turned to 180 degrees
- moved C14 1.35 mm to (87.8, 104.9)
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Connections:
- 0101 pad 2: Net-(LED10-Pad2) -> SPI
- 1000 pad 4: SPI -> (no net)
- C14 pad 1: VSS -> Net-(C14-Pad1)
Routing:
- net IO0: track 3.94 -> 72.0 mm, vias 0 -> 1
- net SPI: track 34.5 -> 83.1 mm
- net IO27: track 55.1 -> 78.1 mm
- net VDD: track 96.4 -> 76.3 mm, vias 28 -> 27
- net VSS: track 49.5 -> 58.5 mm, vias 3 -> 2
- net P2: track 57.9 -> 62.9 mm
- net IO13: track 8.96 -> 13.2 mm, vias 0 -> 2
- net VDDA: track 40.6 -> 44.1 mm
- net IO35: track 7.59 -> 10.1 mm
- net IO33: track 10.0 -> 12.5 mm, vias 0 -> 2
- net P0: track 20.7 -> 18.4 mm
- net Net-(U1-Pad37): track 0.24 -> 2.43 mm, vias 0 -> 1
- net RX: track 81.3 -> 79.3 mm
- net IO32: track 8.76 -> 10.6 mm
- net Net-(C14-Pad1): track 0.00 -> 1.75 mm
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Other:
- board text added: "IO0"
- board text added: "JLCJLCJLCJLC"
- board text added: "v5"
- board text removed: "v4"
