File: Schematic/Badge/badge.sch (KiCad schematic (older format))
At the start: 50 parts, among them J1 Left2, J10 USB_B_Micro, J11 Penny2, J12 Penny1, J13 Penny0, J14 Power, J4 Serial, J5 Penny3, J7 Right2, J8 Right3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

Commit message: v4, changes to add all of the best chineseium bits I can find
Parts:
- removed U3: MCP73831-2-OT, Package_TO_SOT_SMD:SOT-23-5, symbol Battery_Management:MCP73831-2-OT
- added U3: HX4056, Badge:HX4056, symbol badge-rescue:HX4056
- C14, C17: value 4.7uF -> 10uF
- J10: footprint Connectors_USB:USB_Micro-B_Molex_47346-0001 -> Connectors_USB:USB_Micro-B_Jing
- R2: value 2k -> 1k
Connections:
- net IO27: now also U3.6 (STAT2)
- net RX: now also U1.35 (TXD0); no longer U1.34 (RXD0)
- net TX: now also U1.34 (RXD0); no longer U1.35 (TXD0)
- net VBUS: now also U3.4 (Vin)
- net VDDA: now also U3.5 (BAT)
- net VSS: now also U3.3 (GND), U3.9 (GND)
- net at R2.1: now also U3.2 (ISET)
- net IO22: no longer names the net of U1.36 (IO22)
- net IO23: no longer names the net of U1.37 (IO23)
- no-connect marks 12 -> 15
Other:
- moved on the sheet: C17, R2
Changed lines of the file:
@@
 Wire Wire Line
 	6100 3850 6000 3850
-Text GLabel 9650 3600 2    60   Input ~ 0
-IO23
-Text GLabel 9650 3700 2    60   Input ~ 0
-IO22
+Text GLabel 9650 3900 2    60   Input ~ 0
+TX
 Text GLabel 9650 3800 2    60   Input ~ 0
-TX
-Text GLabel 9650 3900 2    60   Input ~ 0
 RX
 Text GLabel 9650 4000 2    60   Input ~ 0
@@
 F 0 "J10" H 2305 5867 50  0000 C CNN
 F 1 "USB_B_Micro" H 2305 5776 50  0000 C CNN
-F 2 "Connectors_USB:USB_Micro-B_Molex_47346-0001" H 2400 5350 50  0001 C CNN
+F 2 "Connectors_USB:USB_Micro-B_Jing" H 2400 5350 50  0001 C CNN
 F 3 "~" H 2400 5350 50  0001 C CNN
 	1    2250 5400
@@
 $EndComp
 $Comp
-L Battery_Management:MCP73831-2-OT U3
-U 1 1 5C33362C
-P 3550 5350
-F 0 "U3" H 3550 5800 50  0000 C CNN
-F 1 "MCP73831-2-OT" H 3650 5700 50  0000 C CNN
-F 2 "Package_TO_SOT_SMD:SOT-23-5" H 3600 5100 50  0001 L CIN
-F 3 "http://ww1.microchip.com/downloads/en/DeviceDoc/20001984g.pdf" H 3400 5300 50  0001 C CNN
-	1    3550 5350
-	1    0    0    -1
-$EndComp
-$Comp
 L power:VDDA #PWR027
 U 1 1 5C33B5E7
-P 4400 5250
-F 0 "#PWR027" H 4400 5100 50  0001 C CNN
-F 1 "VDDA" V 4417 5378 50  0000 L CNN
-F 2 "" H 4400 5250 50  0001 C CNN
-F 3 "" H 4400 5250 50  0001 C CNN
-	1    4400 5250
+P 4650 5100
+F 0 "#PWR027" H 4650 4950 50  0001 C CNN
+F 1 "VDDA" V 4667 5228 50  0000 L CNN
+F 2 "" H 4650 5100 50  0001 C CNN
+F 3 "" H 4650 5100 50  0001 C CNN
+	1    4650 5100
 	0    1    1    0
 $EndComp
@@
 L badge-rescue:C C17
 U 1 1 5C33B6A8
-P 4150 5100
-F 0 "C17" H 4265 5146 50  0000 L CNN
-F 1 "4.7uF" H 4265 5055 50  0000 L CNN
-F 2 "Capacitors_SMD:C_0805_HandSoldering" H 4188 4950 50  0001 C CNN
-F 3 "" H 4150 5100 50  0001 C CNN
-	1    4150 5100
-	1    0    0    -1
-$EndComp
-Connection ~ 4150 5250
-Wire Wire Line
-	4150 5250 4400 5250
-Wire Wire Line
-	3950 5250 4150 5250
+P 4400 4950
+F 0 "C17" H 4515 4996 50  0000 L CNN
+F 1 "10uF" H 4515 4905 50  0000 L CNN
+F 2 "Capacitors_SMD:C_0805_HandSoldering" H 4438 4800 50  0001 C CNN
+F 3 "" H 4400 4950 50  0001 C CNN
+	1    4400 4950
+	1    0    0    -1
+$EndComp
+Connection ~ 4400 5100
+Wire Wire Line
+	4400 5100 4650 5100
+Wire Wire Line
+	4200 5100 4400 5100
 $Comp
 L power:VSS #PWR025
 U 1 1 5C33F9EB
-P 4150 4950
-F 0 "#PWR025" H 4150 4800 50  0001 C CNN
-F 1 "VSS" H 4167 5123 50  0000 C CNN
-F 2 "" H 4150 4950 50  0001 C CNN
-F 3 "" H 4150 4950 50  0001 C CNN
-	1    4150 4950
+P 4400 4800
+F 0 "#PWR025" H 4400 4650 50  0001 C CNN
+F 1 "VSS" H 4417 4973 50  0000 C CNN
+F 2 "" H 4400 4800 50  0001 C CNN
+F 3 "" H 4400 4800 50  0001 C CNN
+	1    4400 4800
 	1    0    0    -1
 $EndComp
@@
 L power:VSS #PWR021
 U 1 1 5C33FAD9
-P 3550 5650
-F 0 "#PWR021" H 3550 5500 50  0001 C CNN
-F 1 "VSS" H 3568 5823 50  0000 C CNN
-F 2 "" H 3550 5650 50  0001 C CNN
-F 3 "" H 3550 5650 50  0001 C CNN
-	1    3550 5650
+P 4200 5400
+F 0 "#PWR021" H 4200 5250 50  0001 C CNN
+F 1 "VSS" H 4218 5573 50  0000 C CNN
+F 2 "" H 4200 5400 50  0001 C CNN
+F 3 "" H 4200 5400 50  0001 C CNN
+	1    4200 5400
 	-1   0    0    1
 $EndComp
@@
 P 2900 4900
 F 0 "C14" H 3015 4946 50  0000 L CNN
-F 1 "4.7uF" H 3015 4855 50  0000 L CNN
+F 1 "10uF" H 3015 4855 50  0000 L CNN
 F 2 "Capacitors_SMD:C_0805_HandSoldering" H 2938 4750 50  0001 C CNN
 F 3 "" H 2900 4900 50  0001 C CNN
@@
 Connection ~ 2900 5050
 Wire Wire Line
-	2900 5050 3050 5050
+	2900 5050 2950 5050
 $Comp
 L power:VSS #PWR019
@@
 L power:VBUS #PWR020
 U 1 1 5C34F2AC
-P 3050 5050
-F 0 "#PWR020" H 3050 4900 50  0001 C CNN
-F 1 "VBUS" H 3065 5223 50  0000 C CNN
-F 2 "" H 3050 5050 50  0001 C CNN
-F 3 "" H 3050 5050 50  0001 C CNN
-	1    3050 5050
-	-1   0    0    1
-$EndComp
-Connection ~ 3050 5050
-Wire Wire Line
-	3050 5050 3550 5050
+P 2950 5050
+F 0 "#PWR020" H 2950 4900 50  0001 C CNN
+F 1 "VBUS" H 2965 5223 50  0000 C CNN
+F 2 "" H 2950 5050 50  0001 C CNN
+F 3 "" H 2950 5050 50  0001 C CNN
+	1    2950 5050
+	-1   0    0    1
+$EndComp
 $Comp
 L power:VBUS #PWR022
@@
 L badge-rescue:R R2
 U 1 1 5C37B5B5
-P 3000 5450
-F 0 "R2" V 3100 5450 50  0000 C CNN
-F 1 "2k" V 3200 5450 50  0000 C CNN
-F 2 "Resistors_SMD:R_0805_HandSoldering" V 2930 5450 50  0001 C CNN
-F 3 "" H 3000 5450 50  0001 C CNN
-	1    3000 5450
-	0    1    1    0
+P 4350 5200
+F 0 "R2" V 4450 5200 50  0000 C CNN
+F 1 "1k" V 4550 5200 50  0000 C CNN
+F 2 "Resistors_SMD:R_0805_HandSoldering" V 4280 5200 50  0001 C CNN
+F 3 "" H 4350 5200 50  0001 C CNN
+	1    4350 5200
+	0    -1   1    0
 $EndComp
 $Comp
 L power:VSS #PWR030
 U 1 1 5C37B705
-P 2850 5450
-F 0 "#PWR030" H 2850 5300 50  0001 C CNN
-F 1 "VSS" H 2868 5623 50  0000 C CNN
-F 2 "" H 2850 5450 50  0001 C CNN
-F 3 "" H 2850 5450 50  0001 C CNN
-	1    2850 5450
-	-1   0    0    1
-$EndComp
-Text GLabel 3950 5450 2    50   Input ~ 0
+P 4500 5200
+F 0 "#PWR030" H 4500 5050 50  0001 C CNN
+F 1 "VSS" H 4518 5373 50  0000 C CNN
+F 2 "" H 4500 5200 50  0001 C CNN
+F 3 "" H 4500 5200 50  0001 C CNN
+	1    4500 5200
+	1    0    0    1
+$EndComp
+Text GLabel 3300 5200 0    50   Input ~ 0
 IO27
 NoConn ~ 2550 5600
@@
 	0    -1   -1   0
 $EndComp
+$Comp
+L badge-rescue:HX4056 U3
+U 1 1 5C6DE973
+P 3800 5200
+F 0 "U3" H 3750 5525 50  0000 C CNN
+F 1 "HX4056" H 3750 5434 50  0000 C CNN
+F 2 "Badge:HX4056" H 3700 5200 50  0001 C CNN
+F 3 "" H 3700 5200 50  0001 C CNN
+	1    3800 5200
+	1    0    0    -1
+$EndComp
+Connection ~ 2950 5050
+Wire Wire Line
+	3300 5050 3300 5100
+Wire Wire Line
+	2950 5050 3300 5050
+$Comp
+L power:VSS #PWR05
+U 1 1 5C7050D7
+P 3300 5400
+F 0 "#PWR05" H 3300 5250 50  0001 C CNN
+F 1 "VSS" H 3318 5573 50  0000 C CNN
+F 2 "" H 3300 5400 50  0001 C CNN
+F 3 "" H 3300 5400 50  0001 C CNN
+	1    3300 5400
+	-1   0    0    1
+$EndComp
+NoConn ~ 3300 5300
+NoConn ~ 9650 3600
+NoConn ~ 9650 3700
+Connection ~ 7800 5050
 $EndSCHEMATC

Commit message: v5 arrived
Parts:
- added J2: Conn_02x03_Odd_Even, symbol Connector_Generic:Conn_02x03_Odd_Even
- added R5: 1.5, Resistors_SMD:R_0805, symbol Device:R_Small
Connections:
- net SPI: now also LED10.2 (DOUT); no longer LED1.4 (DIN)
- net VSS: now also R5.1; no longer C14.1
- new net: C14.1, R5.2
Other:
- moved on the sheet: J1, J11, J12, J13, J14, J4, J5, J7, J8, J9
Changed lines of the file:
@@
 Wire Wire Line
 	10050 1300 10050 1100
-Connection ~ 10050 1100
 Wire Wire Line
 	10850 1400 10850 1600
-Connection ~ 10850 1600
-Wire Wire Line
-	1050 1400 1050 1800
-Text GLabel 1050 1800 3    60   Input ~ 0
+Text GLabel 10950 1850 3    60   Input ~ 0
 SPI
 Wire Wire Line
@@
 L badge-rescue:Conn_01x02 J4
 U 1 1 5AD6B1DD
-P 2100 2650
-F 0 "J4" H 2100 2750 50  0000 C CNN
-F 1 "Serial" H 2100 2450 50  0000 C CNN
-F 2 "Wire_Pads:SolderWirePad_2x_1mmDrill" H 2100 2650 50  0001 C CNN
-F 3 "" H 2100 2650 50  0001 C CNN
-	1    2100 2650
-	-1   0    0    1
-$EndComp
-Text GLabel 2300 2550 2    60   Input ~ 0
+P 1100 4450
+F 0 "J4" H 1100 4550 50  0000 C CNN
+F 1 "Serial" H 1100 4250 50  0000 C CNN
+F 2 "Wire_Pads:SolderWirePad_2x_1mmDrill" H 1100 4450 50  0001 C CNN
+F 3 "" H 1100 4450 50  0001 C CNN
+	1    1100 4450
+	-1   0    0    1
+$EndComp
+Text GLabel 1300 4350 2    60   Input ~ 0
 TX
-Text GLabel 2300 2650 2    60   Input ~ 0
+Text GLabel 1300 4450 2    60   Input ~ 0
 RX
-Text GLabel 1350 2950 2    60   Input ~ 0
+Text GLabel 1300 2300 2    60   Input ~ 0
 IO34
-Text GLabel 1350 3050 2    60   Input ~ 0
+Text GLabel 1300 2400 2    60   Input ~ 0
 IO35
-Text GLabel 1350 3150 2    60   Input ~ 0
+Text GLabel 1300 2500 2    60   Input ~ 0
 IO32
-Text GLabel 1350 3250 2    60   Input ~ 0
+Text GLabel 1300 2600 2    60   Input ~ 0
 IO33
 $Comp
 L badge-rescue:Conn_01x04 J1
 U 1 1 5AD7CE57
-P 1150 3150
-F 0 "J1" H 1150 3350 50  0000 C CNN
-F 1 "Left2" H 1150 2850 50  0000 C CNN
-F 2 "Pin_Headers:Pin_Header_Straight_1x04_Pitch2.54mm" H 1150 3150 50  0001 C CNN
-F 3 "" H 1150 3150 50  0001 C CNN
-	1    1150 3150
+P 1100 2500
+F 0 "J1" H 1100 2700 50  0000 C CNN
+F 1 "Left2" H 1100 2200 50  0000 C CNN
+F 2 "Pin_Headers:Pin_Header_Straight_1x04_Pitch2.54mm" H 1100 2500 50  0001 C CNN
+F 3 "" H 1100 2500 50  0001 C CNN
+	1    1100 2500
 	-1   0    0    1
 $EndComp
@@
 L badge-rescue:Conn_01x01 J7
 U 1 1 5AD7DD02
-P 2900 2950
-F 0 "J7" H 2900 3050 50  0000 C CNN
-F 1 "Right2" H 2900 2850 50  0000 C CNN
-F 2 "Wire_Pads:SolderWirePad_single_1mmDrill" H 2900 2950 50  0001 C CNN
-F 3 "" H 2900 2950 50  0001 C CNN
-	1    2900 2950
-	-1   0    0    1
-$EndComp
-Text GLabel 3100 2950 2    60   Input ~ 0
+P 1100 3650
+F 0 "J7" H 1100 3750 50  0000 C CNN
+F 1 "Right2" H 1100 3550 50  0000 C CNN
+F 2 "Wire_Pads:SolderWirePad_single_1mmDrill" H 1100 3650 50  0001 C CNN
+F 3 "" H 1100 3650 50  0001 C CNN
+	1    1100 3650
+	-1   0    0    1
+$EndComp
+Text GLabel 1300 3650 2    60   Input ~ 0
 IO21
-Text GLabel 3100 3300 2    60   Input ~ 0
+Text GLabel 1300 2900 2    60   Input ~ 0
 IO19
-Text GLabel 3100 3400 2    60   Input ~ 0
+Text GLabel 1300 3000 2    60   Input ~ 0
 IO18
-Text GLabel 3100 3500 2    60   Input ~ 0
+Text GLabel 1300 3100 2    60   Input ~ 0
 IO5
-Text GLabel 3100 3600 2    60   Input ~ 0
+Text GLabel 1300 3200 2    60   Input ~ 0
 IO17
-Text GLabel 3100 3700 2    60   Input ~ 0
+Text GLabel 1300 3300 2    60   Input ~ 0
 IO16
 $Comp
 L badge-rescue:Conn_01x05 J8
 U 1 1 5AD7E240
-P 2900 3500
-F 0 "J8" H 2900 3800 50  0000 C CNN
-F 1 "Right3" H 2900 3200 50  0000 C CNN
-F 2 "Pin_Headers:Pin_Header_Straight_1x05_Pitch2.54mm" H 2900 3500 50  0001 C CNN
-F 3 "" H 2900 3500 50  0001 C CNN
-	1    2900 3500
+P 1100 3100
+F 0 "J8" H 1100 3400 50  0000 C CNN
+F 1 "Right3" H 1100 2800 50  0000 C CNN
+F 2 "Pin_Headers:Pin_Header_Straight_1x05_Pitch2.54mm" H 1100 3100 50  0001 C CNN
+F 3 "" H 1100 3100 50  0001 C CNN
+	1    1100 3100
 	-1   0    0    1
 $EndComp
@@
 L badge-rescue:Conn_01x01 J9
 U 1 1 5AD7E2BD
-P 2900 4000
-F 0 "J9" H 2900 4100 50  0000 C CNN
-F 1 "Right4" H 2900 3900 50  0000 C CNN
-F 2 "Wire_Pads:SolderWirePad_single_1mmDrill" H 2900 4000 50  0001 C CNN
-F 3 "" H 2900 4000 50  0001 C CNN
-	1    2900 4000
-	-1   0    0    1
-$EndComp
-Text GLabel 3100 4000 2    60   Input ~ 0
+P 1100 3950
+F 0 "J9" H 1100 4050 50  0000 C CNN
+F 1 "Right4" H 1100 3850 50  0000 C CNN
+F 2 "Wire_Pads:SolderWirePad_single_1mmDrill" H 1100 3950 50  0001 C CNN
+F 3 "" H 1100 3950 50  0001 C CNN
+	1    1100 3950
+	-1   0    0    1
+$EndComp
+Text GLabel 1300 3950 2    60   Input ~ 0
 IO0
 $Comp
@@
 Connection ~ 5000 1600
 Connection ~ 6000 1600
-NoConn ~ 10850 1300
 Wire Wire Line
 	9000 1300 9050 1300
@@
 L badge-rescue:Conn_01x01 J13
 U 1 1 5AF8C2A5
-P 950 6000
-F 0 "J13" H 950 6100 50  0000 C CNN
-F 1 "Penny0" H 950 5900 50  0000 C CNN
-F 2 "Wire_Pads:Penny" H 950 6000 50  0001 C CNN
-F 3 "" H 950 6000 50  0001 C CNN
-	1    950  6000
+P 1100 6650
+F 0 "J13" H 1100 6750 50  0000 C CNN
+F 1 "Penny0" H 1100 6550 50  0000 C CNN
+F 2 "Wire_Pads:Penny" H 1100 6650 50  0001 C CNN
+F 3 "" H 1100 6650 50  0001 C CNN
+	1    1100 6650
 	-1   0    0    1
 $EndComp
@@
 L badge-rescue:Conn_01x01 J12
 U 1 1 5AF8C41B
-P 950 5700
-F 0 "J12" H 950 5800 50  0000 C CNN
-F 1 "Penny1" H 950 5600 50  0000 C CNN
-F 2 "Wire_Pads:Penny" H 950 5700 50  0001 C CNN
-F 3 "" H 950 5700 50  0001 C CNN
-	1    950  5700
+P 1100 6350
+F 0 "J12" H 1100 6450 50  0000 C CNN
+F 1 "Penny1" H 1100 6250 50  0000 C CNN
+F 2 "Wire_Pads:Penny" H 1100 6350 50  0001 C CNN
+F 3 "" H 1100 6350 50  0001 C CNN
+	1    1100 6350
 	-1   0    0    1
 $EndComp
@@
 L badge-rescue:Conn_01x01 J5
 U 1 1 5AF8C77A
-P 950 5100
-F 0 "J5" H 950 5200 50  0000 C CNN
-F 1 "Penny3" H 950 5000 50  0000 C CNN
-F 2 "Wire_Pads:Penny" H 950 5100 50  0001 C CNN
-F 3 "" H 950 5100 50  0001 C CNN
-	1    950  5100
+P 1100 5750
+F 0 "J5" H 1100 5850 50  0000 C CNN
+F 1 "Penny3" H 1100 5650 50  0000 C CNN
+F 2 "Wire_Pads:Penny" H 1100 5750 50  0001 C CNN
+F 3 "" H 1100 5750 50  0001 C CNN
+	1    1100 5750
 	-1   0    0    1
 $EndComp
@@
 L badge-rescue:Conn_01x01 J11
 U 1 1 5AF8C780
-P 950 5400
-F 0 "J11" H 950 5500 50  0000 C CNN
-F 1 "Penny2" H 950 5300 50  0000 C CNN
-F 2 "Wire_Pads:Penny" H 950 5400 50  0001 C CNN
-F 3 "" H 950 5400 50  0001 C CNN
-	1    950  5400
-	-1   0    0    1
-$EndComp
-Text GLabel 1150 5100 2    60   Input ~ 0
+P 1100 6050
+F 0 "J11" H 1100 6150 50  0000 C CNN
+F 1 "Penny2" H 1100 5950 50  0000 C CNN
+F 2 "Wire_Pads:Penny" H 1100 6050 50  0001 C CNN
+F 3 "" H 1100 6050 50  0001 C CNN
+	1    1100 6050
+	-1   0    0    1
+$EndComp
+Text GLabel 1300 5750 2    60   Input ~ 0
 P3
-Text GLabel 1150 5400 2    60   Input ~ 0
+Text GLabel 1300 6050 2    60   Input ~ 0
 P2
-Text GLabel 1150 6000 2    60   Input ~ 0
+Text GLabel 1300 6650 2    60   Input ~ 0
 P0
-Text GLabel 1150 5700 2    60   Input ~ 0
+Text GLabel 1300 6350 2    60   Input ~ 0
 P1
 $Comp
@@
 L badge-rescue:Conn_01x02 J14
 U 1 1 5AF927B2
-P 3900 2650
-F 0 "J14" H 3900 2750 50  0000 C CNN
-F 1 "Power" H 3900 2450 50  0000 C CNN
-F 2 "Wire_Pads:SolderWirePad_2x_1mmDrill" H 3900 2650 50  0001 C CNN
-F 3 "" H 3900 2650 50  0001 C CNN
-	1    3900 2650
+P 1100 5400
+F 0 "J14" H 1100 5500 50  0000 C CNN
+F 1 "Power" H 1100 5200 50  0000 C CNN
+F 2 "Wire_Pads:SolderWirePad_2x_1mmDrill" H 1100 5400 50  0001 C CNN
+F 3 "" H 1100 5400 50  0001 C CNN
+	1    1100 5400
 	-1   0    0    1
 $EndComp
@@
 L power:VSS #PWR013
 U 1 1 5AF92923
-P 4100 2550
-F 0 "#PWR013" H 4100 2400 50  0001 C CNN
-F 1 "VSS" H 4100 2700 50  0000 C CNN
-F 2 "" H 4100 2550 50  0001 C CNN
-F 3 "" H 4100 2550 50  0001 C CNN
-	1    4100 2550
+P 1300 5300
+F 0 "#PWR013" H 1300 5150 50  0001 C CNN
+F 1 "VSS" H 1300 5450 50  0000 C CNN
+F 2 "" H 1300 5300 50  0001 C CNN
+F 3 "" H 1300 5300 50  0001 C CNN
+	1    1300 5300
 	1    0    0    -1
 $EndComp
@@
 L power:VDD #PWR014
 U 1 1 5AF92987
-P 4100 2650
-F 0 "#PWR014" H 4100 2500 50  0001 C CNN
-F 1 "VDD" H 4100 2800 50  0000 C CNN
-F 2 "" H 4100 2650 50  0001 C CNN
-F 3 "" H 4100 2650 50  0001 C CNN
-	1    4100 2650
+P 1300 5400
+F 0 "#PWR014" H 1300 5250 50  0001 C CNN
+F 1 "VDD" H 1300 5550 50  0000 C CNN
+F 2 "" H 1300 5400 50  0001 C CNN
+F 3 "" H 1300 5400 50  0001 C CNN
+	1    1300 5400
 	0    1    1    0
 $EndComp
@@
 	9850 1600 10000 1600
 Wire Wire Line
-	10050 1100 10950 1100
-Wire Wire Line
-	10850 1600 10950 1600
-Wire Wire Line
 	7550 3400 7550 3350
 Wire Wire Line
@@
 L power:VSS #PWR019
 U 1 1 5C34477D
-P 2900 4750
-F 0 "#PWR019" H 2900 4600 50  0001 C CNN
-F 1 "VSS" H 2917 4923 50  0000 C CNN
-F 2 "" H 2900 4750 50  0001 C CNN
-F 3 "" H 2900 4750 50  0001 C CNN
-	1    2900 4750
+P 2900 4450
+F 0 "#PWR019" H 2900 4300 50  0001 C CNN
+F 1 "VSS" H 2917 4623 50  0000 C CNN
+F 2 "" H 2900 4450 50  0001 C CNN
+F 3 "" H 2900 4450 50  0001 C CNN
+	1    2900 4450
 	1    0    0    -1
 $EndComp
@@
 NoConn ~ 9650 3600
 NoConn ~ 9650 3700
-Connection ~ 7800 5050
+$Comp
+L Connector_Generic:Conn_02x03_Odd_Even J2
+U 1 1 5C7F054A
+P 4800 3800
+F 0 "J2" H 4850 4117 50  0000 C CNN
+F 1 "Conn_02x03_Odd_Even" H 4850 4026 50  0000 C CNN
+F 2 "" H 4800 3800 50  0001 C CNN
+F 3 "~" H 4800 3800 50  0001 C CNN
+	1    4800 3800
+	1    0    0    -1
+$EndComp
+Wire Wire Line
+	10850 1300 10950 1300
+Wire Wire Line
+	10950 1300 10950 1850
+NoConn ~ 1050 1400
+$Comp
+L Device:R_Small R5
+U 1 1 5C9B4547
+P 2900 4600
+F 0 "R5" H 2959 4646 50  0000 L CNN
+F 1 "1.5" H 2959 4555 50  0000 L CNN
+F 2 "Resistors_SMD:R_0805" H 2900 4600 50  0001 C CNN
+F 3 "~" H 2900 4600 50  0001 C CNN
+	1    2900 4600
+	1    0    0    -1
+$EndComp
+Wire Wire Line
+	2900 4500 2900 4450
+Wire Wire Line
+	2900 4750 2900 4700
 $EndSCHEMATC
