File: Schematic/Lid/lid.kicad_pcb (KiCad board)
At the start: 2 copper layers, 90.5 x 57.7 mm, 6 parts

Commit message: v5 arrived
Parts:
- removed the G*** at (150.5, 93.5)
- added ?: , Badge:Bsides_InProgress, F.Cu at (144.4, 92.2)
- added ?: , Badge:Iowa, F.Cu at (171.4, 111.8)
Other:
- outline, holes or cut-outs redrawn
- board text added: "JLCJLCJLCJLC"
